File: pcb.sch (KiCad schematic (older format))
At the start: 81 parts, among them J1 USB_mini_B, K1 7, K10 6, K11 3, K12 EQUAL, K13 DEVIDE, K14 *, K15 -, K16 +, K2 4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

Commit message: wiring
Connections:
- net col1: now also U1.30 (PB6); no longer U1.31 (PC6)
- net col2: now also U1.31 (PC6); no longer U1.30 (PB6)
- net col3: now also U1.28 (PB4); no longer U1.29 (PB5)
- net col4: now also U1.29 (PB5); no longer U1.28 (PB4)
- net rgb2: now also U1.38 (PF5); no longer U1.36 (PF7)
- net rgb4: now also U1.36 (PF7); no longer U1.38 (PF5)
Changed lines of the file:
@@
 LIBS:mkl27z256vfm4
 LIBS:mx1a-simple
-LIBS:ws2812b
 LIBS:pcb-cache
 EELAYER 25 0
@@
 Text Label 3500 2800 2    60   ~ 0
 row3
+Text Label 5950 2300 0    60   ~ 0
+col1
 Text Label 5950 2200 0    60   ~ 0
-col1
-Text Label 5950 2300 0    60   ~ 0
 col2
-Text Label 5950 2400 0    60   ~ 0
+Text Label 5950 2500 0    60   ~ 0
 col3
 $Comp
@@
 	0    -1   -1   0
 $EndComp
-Text Label 5950 2500 0    60   ~ 0
+Text Label 5950 2400 0    60   ~ 0
 col4
 Text Label 3500 2900 2    60   ~ 0
@@
 Text Label 5950 1400 0    60   ~ 0
 rgb1
-Text Label 5950 1700 0    60   ~ 0
+Text Label 5950 1500 0    60   ~ 0
 rgb2
 Text Label 5950 1600 0    60   ~ 0
 rgb3
-Text Label 5950 1500 0    60   ~ 0
+Text Label 5950 1700 0    60   ~ 0
 rgb4
 Text Label 14400 3700 0    60   ~ 0
@@
 Connection ~ 13850 6950
 Wire Wire Line
-	5950 2500 5800 2500
-Wire Wire Line
-	5800 2400 5950 2400
-Wire Wire Line
-	5950 2300 5800 2300
-Wire Wire Line
-	5800 2200 5950 2200
-Wire Wire Line
 	3500 2900 3650 2900
 Wire Wire Line
@@
 Connection ~ 2900 2550
 Wire Wire Line
+	5800 1600 5950 1600
+Wire Wire Line
+	5950 2200 5800 2200
+Wire Wire Line
+	5800 2300 5950 2300
+Wire Wire Line
+	5950 2400 5800 2400
+Wire Wire Line
+	5800 2500 5950 2500
+Wire Wire Line
 	5950 1500 5800 1500
 Wire Wire Line
-	5800 1600 5950 1600
-Wire Wire Line
-	5950 1700 5800 1700
+	5800 1700 5950 1700
 $EndSCHEMATC

Commit message: re wiring
Connections:
- net row1: now also U1.39 (PF4); no longer U1.18 (PD0/INT0)
- net row2: now also U1.38 (PF5); no longer U1.19 (PD1/INT1)
- net row3: now also U1.37 (PF6); no longer U1.20 (PD2/RXD1)
- net row4: now also U1.36 (PF7); no longer U1.21 (PD3/TXD1)
- net rgb: now reaches U1.40 (PF1)
- net rgb: now also LED1.4 (DIN)
- net at LED4.2 (DOUT): now also LED5.4 (DIN)
- net at LED8.2 (DOUT): now also LED9.4 (DIN)
- net at LED12.2 (DOUT): now also LED13.4 (DIN)
- removed net rgb1: LED1.4 (DIN), U1.39 (PF4)
- removed net rgb2: LED5.4 (DIN), U1.38 (PF5)
- removed net rgb3: LED9.4 (DIN), U1.37 (PF6)
- removed net rgb4: LED13.4 (DIN), U1.36 (PF7)
Changed lines of the file:
@@
 LIBS:mkl27z256vfm4
 LIBS:mx1a-simple
+LIBS:ws2812b
 LIBS:pcb-cache
 EELAYER 25 0
@@
 Text Label 5800 4150 0    60   ~ 0
 col4
-Text Label 3500 2600 2    60   ~ 0
+Text Label 5950 1400 0    60   ~ 0
 row1
-Text Label 3500 2700 2    60   ~ 0
+Text Label 5950 1500 0    60   ~ 0
 row2
-Text Label 3500 2800 2    60   ~ 0
+Text Label 5950 1600 0    60   ~ 0
 row3
 Text Label 5950 2300 0    60   ~ 0
@@
 Text Label 5950 2400 0    60   ~ 0
 col4
-Text Label 3500 2900 2    60   ~ 0
+Text Label 5950 1700 0    60   ~ 0
 row4
-Text Label 5950 1400 0    60   ~ 0
-rgb1
-Text Label 5950 1500 0    60   ~ 0
-rgb2
-Text Label 5950 1600 0    60   ~ 0
-rgb3
-Text Label 5950 1700 0    60   ~ 0
-rgb4
+Text Label 5950 1300 0    60   ~ 0
+rgb
 Text Label 14400 3700 0    60   ~ 0
-rgb1
-Text Label 14400 5050 0    60   ~ 0
-rgb2
-Text Label 14400 6300 0    60   ~ 0
-rgb3
-Text Label 14400 7650 0    60   ~ 0
-rgb4
+rgb
 $Comp
 L C C11
@@
 Connection ~ 13850 6950
 Wire Wire Line
-	3500 2900 3650 2900
-Wire Wire Line
-	3650 2800 3500 2800
-Wire Wire Line
-	3500 2700 3650 2700
-Wire Wire Line
-	3650 2600 3500 2600
-Wire Wire Line
-	5800 1400 5950 1400
-Wire Wire Line
 	12850 4100 12400 4100
 Wire Wire Line
@@
 	9150 7650 8800 7650
 Wire Wire Line
-	13850 7650 14400 7650
-Wire Wire Line
-	13850 6300 14400 6300
-Wire Wire Line
 	12850 6700 12450 6700
 Wire Wire Line
@@
 Wire Wire Line
 	13850 3700 14400 3700
-Wire Wire Line
-	14400 5050 13850 5050
 Wire Wire Line
 	12850 5450 12450 5450
@@
 Connection ~ 2900 2550
 Wire Wire Line
-	5800 1600 5950 1600
-Wire Wire Line
 	5950 2200 5800 2200
 Wire Wire Line
@@
 	5800 2500 5950 2500
 Wire Wire Line
-	5950 1500 5800 1500
+	7800 4100 7800 4600
+Wire Wire Line
+	7800 4600 13850 4600
+Wire Wire Line
+	13850 4600 13850 5050
+Wire Wire Line
+	7800 5450 7800 5900
+Wire Wire Line
+	7800 5900 13850 5900
+Wire Wire Line
+	13850 5900 13850 6300
+Wire Wire Line
+	7800 6700 7800 7300
+Wire Wire Line
+	7800 7300 13850 7300
+Wire Wire Line
+	13850 7300 13850 7650
+Wire Wire Line
+	5950 1300 5800 1300
+Wire Wire Line
+	5950 1400 5800 1400
+Wire Wire Line
+	5800 1500 5950 1500
+Wire Wire Line
+	5950 1600 5800 1600
 Wire Wire Line
 	5800 1700 5950 1700
