File: pcb.kicad_pcb (KiCad board)
At the start: 2 copper layers, 75.9 x 75.9 mm, 81 parts, among them J1 USB_mini_B, K1 7, K10 6, K11 3, K12 EQUAL, K13 DEVIDE, K14 *, K15 -, K16 +, K2 4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

Commit message: wiring
Parts:
- moved C23 10.4 mm to (110.1, 95.1)
- moved C22 10.4 mm to (91.1, 95.1)
- moved C21 10.4 mm to (72.1, 95.1)
- moved C20 10.4 mm to (53.1, 95.1), turned to 270 degrees
- moved C19 10.4 mm to (110.1, 76.1)
- moved C18 10.4 mm to (91.1, 76.1)
- moved C15 10.3 mm to (110.1, 57.1)
Connections:
- U1 pad 28: /col4 -> /col3
- U1 pad 29: /col3 -> /col4
- U1 pad 30: /col2 -> /col1
- U1 pad 31: /col1 -> /col2
- U1 pad 36: /rgb2 -> /rgb4
- U1 pad 38: /rgb4 -> /rgb2
Routing:
- net GND: track 92.6 -> 259.2 mm, vias 5 -> 13
- net VCC: track 101.3 -> 208.2 mm, vias 2 -> 4
- net /col4: track 57.1 -> 106.8 mm, vias 0 -> 3
- net /col1: track 57.1 -> 98.3 mm, vias 0 -> 3
- net /col3: track 61.0 -> 80.2 mm, vias 0 -> 1
- net /col2: track 57.1 -> 71.4 mm, vias 0 -> 1
- net /rgb4: track 77.5 -> 65.8 mm, vias 0 -> 2
- net /rgb3: track 57.2 -> 47.8 mm, vias 0 -> 2
- net /rgb1: track 52.6 -> 48.1 mm
- net Net-(D8-Pad2): track 0.00 -> 3.80 mm
- net /rgb2: track 29.6 -> 30.8 mm

Commit message: re wiring
Parts:
- moved C12 10.4 mm to (53.2, 57.0)
- moved C16 10.4 mm to (53.2, 76.0)
- moved C14 9.65 mm to (91.5, 57.8), turned to 180 degrees
- moved C17 5.68 mm to (73.5, 80.9)
- moved C13 5.34 mm to (58.8, 57.2), turned to 90 degrees
Connections:
- LED1 pad 4: /rgb1 -> /rgb
- LED13 pad 4: /rgb4 -> Net-(LED12-Pad2)
- LED5 pad 4: /rgb2 -> Net-(LED4-Pad2)
- LED9 pad 4: /rgb3 -> Net-(LED8-Pad2)
- U1 pad 18: /row1 -> Net-(U1-Pad18)
- U1 pad 19: /row2 -> Net-(U1-Pad19)
- U1 pad 20: /row3 -> Net-(U1-Pad20)
- U1 pad 21: /row4 -> Net-(U1-Pad21)
- U1 pad 36: /rgb4 -> /row4
- U1 pad 37: /rgb3 -> /row3
- U1 pad 38: /rgb2 -> /row2
- U1 pad 39: /rgb1 -> /row1
- U1 pad 40: Net-(U1-Pad40) -> /rgb
Routing:
- net VCC: track 208.2 -> 392.0 mm, vias 4 -> 9
- net GND: track 259.2 -> 422.7 mm, vias 13 -> 21
- net Net-(LED4-Pad2): track 0.00 -> 94.7 mm, vias 0 -> 2
- net Net-(LED8-Pad2): track 0.00 -> 83.8 mm
- net Net-(LED12-Pad2): track 0.00 -> 81.4 mm, vias 0 -> 2
- net /rgb4: track 65.8 -> 0.00 mm, vias 2 -> 0
- net /rgb: track 0.00 -> 48.3 mm
- net /rgb1: track 48.1 -> 0.00 mm
- net /rgb3: track 47.8 -> 0.00 mm, vias 2 -> 0
- net /rgb2: track 30.8 -> 0.00 mm
- net /row1: track 45.6 -> 70.2 mm, vias 2 -> 4
- net Net-(D1-Pad2): track 1.28 -> 12.8 mm
- net Net-(D5-Pad2): track 1.28 -> 5.04 mm

Commit message: v1 complete
Parts:
- added Poker_oval_hole: VAL**, keyboard_parts:Poker_oval_hole, F.Cu at (38.2, 52.5)
- added Poker_oval_hole: VAL**, keyboard_parts:Poker_oval_hole, F.Cu at (38.2, 90.6)
- added Poker_oval_hole: VAL**, keyboard_parts:Poker_oval_hole, F.Cu at (113.1, 71.6)
- added Poker_oval_hole: VAL**, keyboard_parts:Poker_oval_hole, F.Cu at (113.1, 52.6)
- added Poker_oval_hole: VAL**, keyboard_parts:Poker_oval_hole, F.Cu at (113.1, 91.1)
- added REF**: 5holes, help14_keyboard:5holes, B.Cu at (83.4, 54.1)
- added REF**: 5holes, help14_keyboard:5holes_square, B.Cu at (78.9, 47.3)
- moved D4 8.01 mm to (49.1, 107.6), turned to 180 degrees
- moved D3 1.99 mm to (41.4, 85.5)
Routing:
- net GND: track 422.7 -> 613.4 mm, vias 21 -> 32
- net /row4: track 57.4 -> 48.1 mm
- net VCC: track 392.0 -> 400.2 mm, vias 9 -> 10
- net Net-(U1-Pad18): track 0.00 -> 7.09 mm
- net Net-(U1-Pad19): track 0.00 -> 5.63 mm, vias 0 -> 2
- net Net-(U1-Pad22): track 0.00 -> 4.79 mm, vias 0 -> 2
- net Net-(U1-Pad11): track 0.00 -> 3.75 mm, vias 0 -> 2
- net Net-(U1-Pad9): track 0.00 -> 3.42 mm, vias 0 -> 2
- net Net-(U1-Pad7): track 0.00 -> 3.41 mm
- net Net-(U1-Pad21): track 0.00 -> 3.22 mm, vias 0 -> 2
- net Net-(LED8-Pad2): track 83.8 -> 80.8 mm
- net Net-(U1-Pad12): track 0.00 -> 2.52 mm
- net /col3: track 80.2 -> 77.9 mm
- net Net-(U1-Pad8): track 0.00 -> 1.88 mm
- net Net-(LED4-Pad2): track 94.7 -> 96.5 mm
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- added copper zone on B.Cu, net GND
- added copper zone on F.Cu, net GND
Other:
- board text added: "RGB BRICK by help-14"
