File: pcb/pcb.kicad_pcb (KiCad board)
At the start: 2 copper layers, 75.9 x 75.9 mm, 88 parts, among them J1 USB_mini_B, K1 7, K10 6, K11 3, K12 EQUAL, K13 DEVIDE, K14 *, K15 -, K16 +, K2 4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

Commit message: rewiring
Parts:
- removed U1: ATMEGA32U4, QFN50P700X700X100-45N:QFN50P700X700X100-45N
- added IC1: 32U2, keyboard_parts:QFP32, B.Cu at (75.1, 51.6)
- moved REF** 67.0 mm to (17.1, 64.1)
- moved C7 66.1 mm to (19.6, 47.6)
- moved REF** 63.0 mm to (16.6, 56.6)
- moved C4 52.3 mm to (30.6, 49.1)
- moved C5 44.1 mm to (24.6, 60.1)
- moved C3 41.3 mm to (29.6, 61.6)
- moved C6 40.5 mm to (25.6, 55.1)
- moved R2 5.15 mm to (75.1, 63.1), turned to 90 degrees
- moved C24 4.00 mm to (73.8, 43.6), turned to 270 degrees
- moved R1 2.00 mm to (72.6, 65.6), turned to 90 degrees
- moved R3 1.65 mm to (75.6, 43.6)
- moved R4 1.62 mm to (77.3, 43.6)
Connections:
- J1 pad 5: GND -> Net-(IC1-Pad28)
- J1 pad 6: GND -> Net-(IC1-Pad28)
Routing:
- net /row4: track 48.1 -> 100.6 mm, vias 0 -> 2
- net GND: track 613.4 -> 561.4 mm, vias 32 -> 29
- net /row1: track 71.6 -> 28.6 mm, vias 4 -> 2
- net /col1: track 98.5 -> 61.1 mm, vias 3 -> 0
- net /row3: track 57.9 -> 93.4 mm, vias 0 -> 2
- net Net-(IC1-Pad24): track 26.4 -> 2.55 mm, vias 2 -> 0
- net /row2: track 57.1 -> 78.0 mm, vias 0 -> 2
- net VCC: track 400.2 -> 379.6 mm, vias 10 -> 8
- net Net-(IC1-Pad28): track 0.00 -> 7.54 mm
- net Net-(U1-Pad18): track 7.09 -> 0.00 mm
- net /col3: track 77.9 -> 72.0 mm
- net Net-(U1-Pad19): track 5.63 -> 0.00 mm, vias 2 -> 0
- net Net-(LED4-Pad2): track 96.5 -> 101.7 mm, vias 2 -> 3
- net /col2: track 71.4 -> 66.4 mm, vias 1 -> 2
- net Net-(U1-Pad22): track 4.79 -> 0.00 mm, vias 2 -> 0
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
Commit message: done pcb
Parts:
- removed REF**: 5holes, help14_keyboard:5holes
- removed REF**: 5holes, help14_keyboard:5holes_square
- moved Poker_oval_hole 53.2 mm to (75.5, 109.3), turned to 90 degrees
- moved C7 41.7 mm to (61.1, 51.7)
- moved C5 40.9 mm to (64.6, 51.7), turned to 90 degrees
- moved C3 39.8 mm to (68.2, 51.7), turned to 90 degrees
- moved C6 37.4 mm to (62.8, 51.7), turned to 90 degrees
- moved C4 35.9 mm to (66.4, 51.7), turned to 90 degrees
- moved C14 4.32 mm to (95.9, 57.8)
- moved D12 0.76 mm to (79.3, 105.2)
Routing:
- net /col1: track 61.1 -> 96.3 mm, vias 0 -> 3
- net GND: track 561.4 -> 582.4 mm
- net VCC: track 379.6 -> 395.3 mm
- net Net-(C24-Pad1): track 5.31 -> 0.00 mm
- net /row4: track 100.6 -> 104.0 mm
- net Net-(D12-Pad2): track 3.70 -> 4.31 mm

Commit message: small fix
Parts:
- removed Poker_oval_hole (x5): VAL**, keyboard_parts:Poker_oval_hole
- moved C14 11.1 mm to (105.8, 52.7), turned to 90 degrees
- moved C2 6.28 mm to (101.9, 53.9)
- moved C1 6.18 mm to (101.9, 51.4)
- moved X2 3.59 mm to (94.6, 53.4)
- moved X1 1.80 mm to (89.2, 52.7), turned to 270 degrees
Routing:
- net Net-(C1-Pad1): track 18.0 -> 30.9 mm
- net Net-(C2-Pad1): track 19.9 -> 27.6 mm, vias 0 -> 1
- net VCC: track 395.3 -> 390.6 mm
- net (no net): track 0.00 -> 3.80 mm, vias 0 -> 2
- net GND: track 582.4 -> 585.2 mm, vias 29 -> 26

Commit message: add qnf32
Parts:
- added U2: , pcb:QFN-32-1EP_5x5mm_Pitch0.5mm, B.Cu at (75.1, 51.6)
Routing:
- net /col2: track 66.4 -> 94.9 mm
- net VCC: track 390.6 -> 401.5 mm, vias 8 -> 10
- net GND: track 585.2 -> 591.8 mm, vias 26 -> 27
- net (no net): track 3.80 -> 0.00 mm, vias 2 -> 0
- net /col3: track 72.0 -> 74.9 mm
- net Net-(IC1-Pad24): track 2.55 -> 5.03 mm
- net /rgb: track 48.7 -> 51.1 mm
- net Net-(IC1-Pad25): track 0.00 -> 2.34 mm
- net Net-(C1-Pad1): track 30.9 -> 33.2 mm
- net /row3: track 93.4 -> 95.7 mm
- net Net-(IC1-Pad17): track 0.00 -> 2.29 mm
- net /col4: track 106.6 -> 108.8 mm
- net Net-(IC1-Pad15): track 0.00 -> 2.17 mm
- net Net-(IC1-Pad18): track 0.00 -> 2.17 mm
- net /row2: track 78.0 -> 80.1 mm
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Other:
- board size 75.9 x 75.9 mm -> 76 x 75.9 mm
